File: keyguy2.0/output/pcbs/theguy2.kicad_pcb (KiCad board)
At the start: 2 copper layers, 138.2 x 100.5 mm, 87 parts

Commit message: 2.0 done for real this time
Connections:
- D10 pad 1: P104 -> P010
- D11 pad 1: P009 -> P104
- D12 pad 1: P106 -> P009
- D13 pad 1: P104 -> P010
- D14 pad 1: P009 -> P104
- D15 pad 1: P106 -> P009
- D16 pad 1: P104 -> P010
- D17 pad 1: P009 -> P104
- D18 pad 1: P106 -> P009
- D19 pad 1: P104 -> P010
- D20 pad 1: P009 -> P104
- D21 pad 1: P106 -> P009
- D22 pad 1: P104 -> P010
- D4 pad 1: P010 -> P106
- D5 pad 1: P009 -> P104
- D6 pad 1: P106 -> P009
- D7 pad 1: P104 -> P010
- D8 pad 1: P009 -> P104
- D9 pad 1: P106 -> P009
- LED1 pad 2: P006 -> rgb_matrix_index_bottom
- LED1 pad 4: P006 -> rgb_thumbs_layer_cluster
- LED10 pad 2: P006 -> rgb_matrix_hell_top
- LED10 pad 4: P006 -> rgb_matrix_pinky_top
- LED11 pad 2: P006 -> rgb_matrix_pinky_bottom
- LED11 pad 4: P006 -> rgb_matrix_ring_bottom
- LED12 pad 2: P006 -> rgb_matrix_ring_bottom
- LED12 pad 4: P006 -> rgb_matrix_ring_home
- LED13 pad 2: P006 -> rgb_matrix_ring_home
- LED13 pad 4: P006 -> rgb_matrix_ring_top
- LED14 pad 2: P006 -> rgb_matrix_middle_home
- LED14 pad 4: P006 -> rgb_matrix_middle_bottom
- LED15 pad 2: P006 -> rgb_matrix_middle_top
- LED15 pad 4: P006 -> rgb_matrix_middle_home
- LED16 pad 2: P006 -> rgb_matrix_ring_top
- LED16 pad 4: P006 -> rgb_matrix_middle_top
- LED17 pad 2: P006 -> rgb_thumbs_space_cluster
- LED17 pad 4: P006 -> rgb_matrix_index_bottom
- LED18 pad 2: P006 -> rgb_matrix_index_bottom
- LED18 pad 4: P006 -> rgb_matrix_index_home
- LED19 pad 2: P006 -> rgb_matrix_index_home
- LED19 pad 4: P006 -> rgb_matrix_index_top
- LED2 pad 2: P006 -> rgb_thumbs_layer_cluster
- LED2 pad 4: P006 -> rgb_thumbs_space_cluster
- LED20 pad 2: P006 -> rgb_matrix_inner_home
- LED20 pad 4: P006 -> rgb_matrix_inner_bottom
- LED21 pad 2: P006 -> rgb_matrix_inner_top
- LED21 pad 4: P006 -> rgb_matrix_inner_home
- LED22 pad 2: P006 -> rgb_matrix_index_top
- LED22 pad 4: P006 -> rgb_matrix_inner_top
- LED23 pad 2: P006 -> rgb_matrix_index_bottom
- LED23 pad 4: P006 -> rgb_thumbs_layer_cluster
- LED24 pad 2: P006 -> rgb_thumbs_layer_cluster
- LED24 pad 4: P006 -> rgb_thumbs_space_cluster
- LED25 pad 2: P006 -> rgb_matrix_inner_bottom
- LED3 pad 2: P006 -> rgb_matrix_inner_bottom
- LED4 pad 2: P006 -> (no net)
- LED4 pad 4: P006 -> rgb_matrix_hell_last
- LED5 pad 2: P006 -> rgb_matrix_hell_last
- LED5 pad 4: P006 -> rgb_matrix_hell_bottom
- LED6 pad 2: P006 -> rgb_matrix_hell_bottom
- LED6 pad 4: P006 -> rgb_matrix_hell_home
- LED7 pad 2: P006 -> rgb_matrix_hell_home
- LED7 pad 4: P006 -> rgb_matrix_hell_top
- LED8 pad 2: P006 -> rgb_matrix_pinky_home
- LED8 pad 4: P006 -> rgb_matrix_pinky_bottom
- LED9 pad 2: P006 -> rgb_matrix_pinky_top
- LED9 pad 4: P006 -> rgb_matrix_pinky_home
- S1 pad 1: P113 -> P029
- S10 pad 1: P029 -> P113
- S11 pad 1: P002 -> P115
- S12 pad 1: P002 -> P115
- S13 pad 1: P002 -> P115
- S14 pad 1: P115 -> P002
- S15 pad 1: P115 -> P002
- S16 pad 1: P115 -> P002
- S17 pad 1: P113 -> P029
- S18 pad 1: P113 -> P029
- S19 pad 1: P113 -> P029
- S2 pad 1: P111 -> P031
- S20 pad 1: P111 -> P031
- S21 pad 1: P111 -> P031
- S22 pad 1: P111 -> P031
- S23 pad 1: P113 -> P029
- S24 pad 1: P111 -> P031
- S25 pad 1: P111 -> P031
- S3 pad 1: P111 -> P031
- S4 pad 1: P031 -> P111
- S5 pad 1: P031 -> P111
- S6 pad 1: P031 -> P111
- S7 pad 1: P031 -> P111
- S8 pad 1: P029 -> P113
- S9 pad 1: P029 -> P113
