File: keyguy2.0/output/pcbs/theguy2.kicad_pcb (KiCad board)
At the start: 2 copper layers, 138.2 x 100.5 mm, 87 parts

Commit message: 2.0 done for real this time
Connections:
- D25 pad 1: P011 -> P106
- D3 pad 1: P011 -> P106

Commit message: 2.0 done for real this time
Connections:
- D1 pad 1: P010 -> P104
- D2 pad 1: P010 -> P104
- D23 pad 1: P010 -> P104
- D24 pad 1: P010 -> P104

Commit message: pcbs wired
Parts:
- removed the ? at (296.4, 135.4)
- removed the ? at (417.0, 105.0)
- removed the ? at (365.0, 116.2)
- removed the ? at (400.0, 57.5)
- removed the ? at (300.0, 44.5)
- removed the ? at (302.0, 91.0)
- removed the ? at (365.0, 74.5)
- removed D1, D2, D3: , ComboDiode
- removed LED1, LED2, LED3: , WS2812B
- removed S1, S2, S3: , PG1350
- added ?: , HOLE_M2_TH, F.Cu at (352.0, 113.3)
- added ?: , HOLE_M2_TH, F.Cu at (300.0, 124.5)
- added ?: , HOLE_M2_TH, F.Cu at (231.4, 143.7)
- added ?: , HOLE_M2_TH, F.Cu at (235.0, 52.8)
- added ?: , HOLE_M2_TH, F.Cu at (300.0, 82.8)
- added ?: , HOLE_M2_TH, F.Cu at (335.0, 65.8)
- added ?: , HOLE_M2_TH, F.Cu at (237.0, 99.3)
- LED10, LED11, LED12, LED13, LED14, LED15, LED16, LED17, LED18, LED19, LED20, LED21, LED22, LED23, LED24, LED25, LED4, LED5, LED6, LED7, LED8, LED9: moved to F.Cu
- moved S23 65.5 mm to (246.1, 113.9)
- moved D23 65.5 mm to (248.9, 121.4)
- moved B1 65.5 mm to (227.0, 97.0)
- moved D10 65.5 mm to (327.0, 65.3)
- moved D11 65.5 mm to (309.0, 99.3)
- moved D12 65.5 mm to (309.0, 82.3)
- moved D13 65.5 mm to (309.0, 65.3)
- moved D14 65.5 mm to (291.0, 99.3)
- moved D15 65.5 mm to (291.0, 82.3)
- moved D16 65.5 mm to (291.0, 65.3)
- moved D17 65.5 mm to (273.0, 99.3)
- moved D18 65.5 mm to (273.0, 82.3)
- moved D19 65.5 mm to (273.0, 65.3)
- moved D20 65.5 mm to (255.0, 99.3)
- moved D21 65.5 mm to (255.0, 82.3)
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Routing:
- net GND: track 0.00 -> 660.5 mm, vias 0 -> 28
- net VCC: track 0.00 -> 579.1 mm, vias 0 -> 32
- net P106: track 0.00 -> 197.2 mm
- net P031: track 0.00 -> 196.7 mm, vias 0 -> 1
- net P104: track 0.00 -> 192.7 mm
- net P029: track 0.00 -> 161.0 mm, vias 0 -> 1
- net P111: track 0.00 -> 156.6 mm, vias 0 -> 1
- net P113: track 0.00 -> 151.9 mm, vias 0 -> 1
- net pos: track 0.00 -> 149.3 mm
- net P010: track 0.00 -> 143.3 mm, vias 0 -> 3
- net P002: track 0.00 -> 140.4 mm, vias 0 -> 1
- net P009: track 0.00 -> 140.4 mm, vias 0 -> 3
- net P006: track 0.00 -> 123.8 mm, vias 0 -> 1
- net P115: track 0.00 -> 122.2 mm, vias 0 -> 1
- net rgb_matrix_index_bottom: track 0.00 -> 87.7 mm, vias 0 -> 3
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Other:
- net class Default removed

Commit message: added a 2.5 for future minor improvements such as correcting screwsize from m2.5 to m2
Parts:
- removed the ? at (352.0, 113.3)
- removed the ? at (300.0, 124.5)
- removed the ? at (231.4, 143.7)
- removed the ? at (235.0, 52.8)
- removed the ? at (300.0, 82.8)
- removed the ? at (335.0, 65.8)
- removed the ? at (237.0, 99.3)
- added ?: , HOLE_M2_TH, F.Cu at (296.4, 135.4)
- added ?: , HOLE_M2_TH, F.Cu at (417.0, 105.0)
- added ?: , HOLE_M2_TH, F.Cu at (365.0, 116.2)
- added ?: , HOLE_M2_TH, F.Cu at (400.0, 57.5)
- added ?: , HOLE_M2_TH, F.Cu at (300.0, 44.5)
- added ?: , HOLE_M2_TH, F.Cu at (302.0, 91.0)
- added ?: , HOLE_M2_TH, F.Cu at (365.0, 74.5)
- added D1: , ComboDiode, F.Cu at (166.1, 113.1)
- added D2: , ComboDiode, F.Cu at (183.0, 119.3)
- added D3: , ComboDiode, F.Cu at (168.8, 132.2)
- added LED1: , WS2812B,  at (167.3, 110.0)
- added LED2: , WS2812B,  at (184.2, 116.2)
- added LED3: , WS2812B,  at (169.9, 129.1)
- added S1: , PG1350, F.Cu at (168.9, 105.6)
- added S2: , PG1350, F.Cu at (185.8, 111.7)
- added S3: , PG1350, F.Cu at (171.5, 124.6)
- LED10, LED11, LED12, LED13, LED14, LED15, LED16, LED17, LED18, LED19, LED20, LED21, LED22, LED23, LED24, LED25, LED4, LED5, LED6, LED7, LED8, LED9: moved to 
- moved S23 65.5 mm to (311.1, 105.6)
- moved D23 65.5 mm to (313.9, 113.1)
- moved B1 65.5 mm to (292.0, 88.7)
- moved D10 65.5 mm to (392.0, 57.0)
- moved D11 65.5 mm to (374.0, 91.0)
- moved D12 65.5 mm to (374.0, 74.0)
- moved D13 65.5 mm to (374.0, 57.0)
- moved D14 65.5 mm to (356.0, 91.0)
- moved D15 65.5 mm to (356.0, 74.0)
- moved D16 65.5 mm to (356.0, 57.0)
- moved D17 65.5 mm to (338.0, 91.0)
- moved D18 65.5 mm to (338.0, 74.0)
- moved D19 65.5 mm to (338.0, 57.0)
- moved D20 65.5 mm to (320.0, 91.0)
- moved D21 65.5 mm to (320.0, 74.0)
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Routing:
- net GND: track 660.5 -> 0.00 mm, vias 28 -> 0
- net VCC: track 579.1 -> 0.00 mm, vias 32 -> 0
- net P106: track 197.2 -> 0.00 mm
- net P031: track 196.7 -> 0.00 mm, vias 1 -> 0
- net P104: track 192.7 -> 0.00 mm
- net P029: track 161.0 -> 0.00 mm, vias 1 -> 0
- net P111: track 156.6 -> 0.00 mm, vias 1 -> 0
- net P113: track 151.9 -> 0.00 mm, vias 1 -> 0
- net pos: track 149.3 -> 0.00 mm
- net P010: track 143.3 -> 0.00 mm, vias 3 -> 0
- net P002: track 140.4 -> 0.00 mm, vias 1 -> 0
- net P009: track 140.4 -> 0.00 mm, vias 3 -> 0
- net P006: track 123.8 -> 0.00 mm, vias 1 -> 0
- net P115: track 122.2 -> 0.00 mm, vias 1 -> 0
- net rgb_matrix_index_bottom: track 87.7 -> 0.00 mm, vias 3 -> 0
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Other:
- net class Default added: clearance 0.2, trace_width 0.25, via_dia 0.8, via_drill 0.4
